Commit message: added gazebo launch file and urdf changes(collision)

File: urdf/arm.urdf (robot description, URDF)
Before this commit: robot arm, 3 links, 2 joints
Links:
- added link world
- link base_link: mass None -> 1.0; geometry collision box size=0.5 0.5 0.1; visual box size=0.5 0.5 0.1
- link link1: mass None -> 1.0; geometry collision cylinder length=0.5 radius=0.05; visual cylinder length=0.5 radius=0.05
- link link2: mass None -> 1.0; geometry collision cylinder length=0.5 radius=0.05; visual cylinder length=0.5 radius=0.05
Joints:
- added joint world_joint: type fixed, parent world, child base_link, origin xyz=0 0 0 rpy=0 0 0
- joint joint1: limit lower=-3.14 upper=3.14 effort=1.0 velocity=1.0 -> lower=-3.14 upper=3.14 effort=100.0 velocity=1.0; origin xyz=0 0 0 rpy=0 0 0 -> xyz=0 0 0.1 rpy=0 0 0
- joint joint2: axis 1 0 0  -> 1 0 0; limit lower=-3.14 upper=3.14 effort=1.0 velocity=1.0 -> lower=-3.14 upper=3.14 effort=100.0 velocity=1.0
