Commit message: added new script to move the object and changes to launch file for bridge.

File: urdf/arm.xacro.urdf (robot description, URDF)
Before this commit: robot arm, 4 links, 3 joints
Links:
- added link camera_link, mass 0.1; collision box size=0.05 0.05 0.05; visual box size=0.05 0.05 0.05
Joints:
- added joint camera_joint: type fixed, parent base_link, child camera_link, origin xyz=0 0 0.5 rpy=0 0 0

Commit message: added camera sensor

File: urdf/arm.xacro.urdf (robot description, URDF)
Before this commit: robot arm, 5 links, 4 joints
Links:
- added link camera_optical_frame
- link camera_link: mass 0.1 -> None; geometry visual box size=0.05 0.1 0.1
Joints:
- added joint camera_optical_joint: type fixed, parent camera_link, child camera_optical_frame, origin xyz=0 0 0 rpy=-1.57 0 -1.57
- joint camera_joint: origin xyz=0 0 0.5 rpy=0 0 0 -> xyz=0.1 0.1 0.07 rpy=0 0 0

Commit message: changes in the urdf for camera orientation

File: urdf/arm.xacro.urdf (robot description, URDF)
Before this commit: robot arm, 6 links, 5 joints
Links:
- removed link camera_optical_frame
Joints:
- removed joint camera_optical_joint
- joint camera_joint: origin xyz=0.1 0.1 0.07 rpy=0 0 0 -> xyz=0.1 0.1 0.1 rpy=0 0 0
